File: eagle/controller-2.brd (EAGLE design)
At the start: 95.2 x 59.7 mm, 24 parts, among them X1 1751248

Commit message: PCB tweaks
Parts:
- removed R11: (no value), rcl:R0805
- added U$1: THECAVE_LOGO_NEW_TOP_SMALL, thecave:NEW_LOGO_SMALL_TOP
- R10: value (none) -> 1R
- R5: value (none) -> 220K
- R6: value (none) -> 330K
- R7: value (none) -> 470K
- R8: value (none) -> 820K
- R9: value (none) -> 100K
Connections:
- net ANALOG: no longer R11.1
- net GND: no longer R11.2
Routing:
- net ANALOG: track 87.7 -> 85.2 mm
- net GND: track 172.2 -> 170.0 mm
Other:
- board text added: "robo-ctrl-2 thecave.cz"
- board text added: "robo-ctrl-2 thecave.cz rev1"
- board text removed: "robo-ctrl-2"
