File: eagle/controller-2.sch (EAGLE design)
At the start: 24 parts, among them X1 1751248

Commit message: PCB tweaks
Parts:
- removed R11: (no value), rcl:R-EU_R0805
- added U$1: THECAVE_LOGO_NEW_TOP_SMALL, thecave:THECAVE_LOGO_NEW_TOP_SMALL
- R10: value (none) -> 1R
- R5: value (none) -> 220K
- R6: value (none) -> 330K
- R7: value (none) -> 470K
- R8: value (none) -> 820K
- R9: value (none) -> 100K
Connections:
- net ANALOG: no longer R11.1
- net GND: no longer R11.2
Other:
- note added: "relies on internal resistive divider in wemos to pull line down"
- moved on the sheet: JP1, LED1, LED2, LED3, LED4, R1, R2, R3, R4, U$5, X1-1, X1-2
