File: eagle/controller.brd (EAGLE design)
At the start: 95.2 x 59.7 mm, 28 parts, among them M1 NANO, X1 1751248

Commit message: PCB tweaks
Parts:
- added U$6: THECAVE_LOGO_NEW_TOP_SMALL, thecave:NEW_LOGO_SMALL_TOP
- moved R1 1.27 mm to (61.0, 26.7), flipped to the top
Routing:
- net N$2: track 10.3 -> 11.5 mm
- net COM_RX: track 18.8 -> 20.1 mm
Other:
- board text added: "robo-ctrl thecave.cz"
- board text added: "robo-ctrl thecave.cz rev1"
