File: eagle/controller.sch (EAGLE design)
At the start: 28 parts, among them M1 NANO, X1 1751248

Commit message: PCB tweaks
Parts:
- added U$6: THECAVE_LOGO_NEW_TOP_SMALL, thecave:THECAVE_LOGO_NEW_TOP_SMALL
Other:
- note added: "short JP1 and JP2 when digital outputs on C4X and C4Y are needed"
